Commit message: gazebosystem changed to gazebosimsystem still i get error

File: Universal_Robots_ROS2_Description/urdf/ur.ros2_control.xacro (robot description, xacro)
@@ -25,5 +25,5 @@
       <hardware>
         <xacro:if value="${sim_gazebo}">
-          <plugin>gazebo_ros2_control/GazeboSystem</plugin>
+          <plugin>gazebo_ros2_control/GazeboSimSystem</plugin>
         </xacro:if>
         <xacro:if value="${sim_ignition}">

File: install/mir_description/share/mir_description/control/mir_ros2_control.urdf.xacro (robot description, xacro)
@@ -4,5 +4,5 @@
         <ros2_control name="GazeboSystem" type="system">
             <hardware>
-            <plugin>gazebo_ros2_control/GazeboSystem</plugin>
+            <plugin>gazebo_ros2_control/GazeboSimSystem</plugin>
             </hardware>
             <joint name="left_wheel_joint">

File: install/mir_description/share/mir_description/urdf/include/mir_250_v1.urdf.xacro (robot description, xacro)
@@ -6,5 +6,5 @@
   <xacro:include filename="$(find mir_description)/urdf/include/wheel.urdf.xacro" />
   <xacro:include filename="$(find mir_description)/urdf/include/caster.urdf.xacro" />
-  <xacro:include filename="$(find realsense2_description)/urdf/_d435i.urdf.xacro"/>
+  <!-- <xacro:include filename="$(find realsense2_description)/urdf/_d435i.urdf.xacro"/> -->
   <xacro:include filename="$(find robotiq_description)/urdf/robotiq_85_gripper.urdf.xacro"/>
   <xacro:property name="deg_to_rad" value="0.017453293" />
@@ -222,5 +222,5 @@
     <xacro:property name="initial_positions_file" default="$(arg initial_positions_file)"/>
     <!-- create link fixed to the "world" -->
-    <link name="world" />
+    <!-- <link name="world" />
     <joint name="world_joint" type="fixed">
       <parent link="${prefix}base_link" />
@@ -228,4 +228,5 @@
       <origin xyz="0.135 0 0.79" rpy="0 0 ${0.5 * pi}" />
     </joint>
+     -->
     <!-- arm -->
     <xacro:ur_robot
@@ -268,5 +269,5 @@
       <origin xyz="0.135 0 0.79" rpy="0 0 ${0.5 * pi}" /> <!--${0.5 * pi}-->         <!-- position robot in the world -->
     </xacro:ur_robot>
-    <link name="${prefix}camera_mount">
+    <!-- <link name="${prefix}camera_mount">
       <visual>
         <origin xyz="0 0 0" rpy="0 0 0" />
@@ -282,13 +283,13 @@
         </geometry>
       </collision>
-    </link>
-    <joint name="${prefix}camera_mount_joint" type="fixed">
+    </link>     -->
+    <!-- <joint name="${prefix}camera_mount_joint" type="fixed">
       <parent link="ur_flange" />
       <child link="${prefix}camera_mount" />
       <origin xyz="0.035 0.05 0.03" rpy="0 ${pi} ${0.5 * pi}" />
-    </joint>
-    <xacro:sensor_d435i parent="ur_flange" name="realsense" use_nominal_extrinsics="true">
+    </joint>  -->
+    <!-- <xacro:sensor_d435i parent="ur_flange" name="realsense" use_nominal_extrinsics="true">
       <origin xyz="0.02 0 -0.061" rpy="${pi} 0 0"/>
-    </xacro:sensor_d435i>
+    </xacro:sensor_d435i> -->
     <!-- <link name="robotiq_coupler">
       <visual>

File: install/mir_description/share/mir_description/urdf/robots/mir.urdf.xacro (robot description, xacro)
@@ -22,57 +22,4 @@
     left_wheel_joint="${prefix}left_wheel_joint"
     right_wheel_joint="${prefix}right_wheel_joint"/>  -->
-  <ros2_control name="GazeboSystem" type="system">
-    <hardware>
-      <plugin>gazebo_ros2_control/GazeboSystem</plugin>
-    </hardware>
-    <joint name="left_wheel_joint">
-      <command_interface name="velocity">
-        <param name="min">-1</param>
-        <param name="max">1</param>
-      </command_interface>
-      <state_interface name="position"/>
-      <state_interface name="velocity"/>
-    </joint>
-    <joint name="right_wheel_joint">
-      <command_interface name="velocity">
-        <param name="min">-1</param>
-        <param name="max">1</param>
-      </command_interface>
-      <state_interface name="position"/>
-      <state_interface name="velocity"/>
-    </joint>
-    <joint name="fl_caster_rotation_joint">
-      <state_interface name="position"/>
-      <state_interface name="velocity"/>
-    </joint>
-    <joint name="fr_caster_rotation_joint">
-      <state_interface name="position"/>
-      <state_interface name="velocity"/>
-    </joint>
-    <joint name="bl_caster_rotation_joint">
-      <state_interface name="position"/>
-      <state_interface name="velocity"/>
-    </joint>
-    <joint name="br_caster_rotation_joint">
-      <state_interface name="position"/>
-      <state_interface name="velocity"/>
-    </joint>
-    <joint name="fl_caster_wheel_joint">
-      <state_interface name="position"/>
-      <state_interface name="velocity"/>
-    </joint>
-    <joint name="fr_caster_wheel_joint">
-      <state_interface name="position"/>
-      <state_interface name="velocity"/>
-    </joint>
-    <joint name="bl_caster_wheel_joint">
-      <state_interface name="position"/>
-      <state_interface name="velocity"/>
-    </joint>
-    <joint name="br_caster_wheel_joint">
-      <state_interface name="position"/>
-      <state_interface name="velocity"/>
-    </joint>
-  </ros2_control>
   <xacro:include filename="$(find mir_description)/control/gazebo_sim_ros2_control.urdf.xacro" />
   <xacro:load_gazebo_sim_ros2_control_plugin/>

File: install/mir_description/share/mir_description/urdf/robots/robot.urdf (robot description, URDF)
Before this commit: robot mir_250, 49 links, 48 joints
Links:
- removed link camera_mount
- removed link realsense_accel_frame
- removed link realsense_accel_optical_frame
- removed link realsense_bottom_screw_frame
- removed link realsense_color_frame
- removed link realsense_color_optical_frame
- removed link realsense_depth_frame
- removed link realsense_depth_optical_frame
- removed link realsense_gyro_frame
- removed link realsense_gyro_optical_frame
- removed link realsense_infra1_frame
- removed link realsense_infra1_optical_frame
- removed link realsense_infra2_frame
- removed link realsense_infra2_optical_frame
- removed link realsense_link
- removed link world
- link ur_base_link_inertia: mass 0.01 -> 4.0
- link ur_forearm_link: mass 0.01 -> 2.275
- link ur_shoulder_link: mass 0.01 -> 3.7
- link ur_upper_arm_link: mass 0.01 -> 8.393
- link ur_wrist_1_link: mass 0.01 -> 1.219
- link ur_wrist_2_link: mass 0.01 -> 1.219
- link ur_wrist_3_link: mass 0.01 -> 0.1879
Joints:
- removed joint camera_mount_joint
- removed joint realsense_accel_joint
- removed joint realsense_accel_optical_joint
- removed joint realsense_color_joint
- removed joint realsense_color_optical_joint
- removed joint realsense_depth_joint
- removed joint realsense_depth_optical_joint
- removed joint realsense_gyro_joint
- removed joint realsense_gyro_optical_joint
- removed joint realsense_infra1_joint
- removed joint realsense_infra1_optical_joint
- removed joint realsense_infra2_joint
- removed joint realsense_infra2_optical_joint
- removed joint realsense_joint
- removed joint realsense_link_joint
- removed joint world_joint

File: mir_robot/mir_description/urdf/robots/robot.urdf (robot description, URDF)
Before this commit: robot mir_250, 49 links, 48 joints
Links:
- removed link camera_mount
- removed link realsense_accel_frame
- removed link realsense_accel_optical_frame
- removed link realsense_bottom_screw_frame
- removed link realsense_color_frame
- removed link realsense_color_optical_frame
- removed link realsense_depth_frame
- removed link realsense_depth_optical_frame
- removed link realsense_gyro_frame
- removed link realsense_gyro_optical_frame
- removed link realsense_infra1_frame
- removed link realsense_infra1_optical_frame
- removed link realsense_infra2_frame
- removed link realsense_infra2_optical_frame
- removed link realsense_link
- removed link world
Joints:
- removed joint camera_mount_joint
- removed joint realsense_accel_joint
- removed joint realsense_accel_optical_joint
- removed joint realsense_color_joint
- removed joint realsense_color_optical_joint
- removed joint realsense_depth_joint
- removed joint realsense_depth_optical_joint
- removed joint realsense_gyro_joint
- removed joint realsense_gyro_optical_joint
- removed joint realsense_infra1_joint
- removed joint realsense_infra1_optical_joint
- removed joint realsense_infra2_joint
- removed joint realsense_infra2_optical_joint
- removed joint realsense_joint
- removed joint realsense_link_joint
- removed joint world_joint
