Commit message: amidst trying to add gripper

File: mir_robot/mir_description/urdf/include/mir_250_v1.urdf.xacro (robot description, xacro)
@@ -292,5 +292,5 @@
       <origin xyz="0.02 0 -0.061" rpy="${pi} 0 0"/>
     </xacro:sensor_d435i> -->
-    <!-- <link name="robotiq_coupler">
+    <link name="robotiq_coupler">
       <visual>
         <geometry>
@@ -323,5 +323,5 @@
     <xacro:robotiq_85_gripper prefix="" parent="robotiq_coupler" >
       <origin xyz="0 0 0.004" rpy="0 ${-pi/2} ${pi}"/>
-    </xacro:robotiq_85_gripper>  -->
+    </xacro:robotiq_85_gripper>
     <!-- Gazebo FT sensor plugin -->
     <!-- <gazebo reference="wrist_3_joint">

File: mir_robot/mir_description/urdf/robots/mir.urdf.xacro (robot description, xacro)
@@ -26,4 +26,6 @@
   <xacro:include filename="$(find mir_description)/control/mir_ros2_control.urdf.xacro"/>
   <xacro:mir_ros2_control/>
+  <xacro:include filename="$(find mir_description)/control/gripper_ros2_control.xacro"/>
+  <xacro:robotiq_gripper_ros2_control/>
   <!-- i am stupid for changing the above to this fromat cuz either the manipultor ius going to have ...... -->
 </robot>

File: mir_robot/mir_description/urdf/robots/robot.urdf (robot description, URDF)
Before this commit: robot mir_250, 33 links, 32 joints
Links:
- added link robotiq_85_base_link, mass 0.636951; collision mesh filename=package://robotiq_description/meshes/collision/robotiq_85_b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; visual mesh filename=package://robotiq_description/meshes/visual/robotiq_85_base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
- added link robotiq_85_left_finger_link, mass 0.027309; collision mesh filename=package://robotiq_description/meshes/collision/robotiq_85_f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; visual mesh filename=package://robotiq_description/meshes/visual/robotiq_85_fing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
- added link robotiq_85_left_finger_tip_link, mass 0.019555; collision mesh filename=package://robotiq_description/meshes/collision/robotiq_85_f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; visual mesh filename=package://robotiq_description/meshes/visual/robotiq_85_fing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
- added link robotiq_85_left_inner_knuckle_link, mass 0.029951; collision mesh filename=package://robotiq_description/meshes/collision/robotiq_85_i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; visual mesh filename=package://robotiq_description/meshes/visual/robotiq_85_inne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
- added link robotiq_85_left_knuckle_link, mass 0.018491; collision mesh filename=package://robotiq_description/meshes/collision/robotiq_85_k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; visual mesh filename=package://robotiq_description/meshes/visual/robotiq_85_knuc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
- added link robotiq_85_right_finger_link, mass 0.027309; collision mesh filename=package://robotiq_description/meshes/collision/robotiq_85_f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; visual mesh filename=package://robotiq_description/meshes/visual/robotiq_85_fing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
- added link robotiq_85_right_finger_tip_link, mass 0.019555; collision mesh filename=package://robotiq_description/meshes/collision/robotiq_85_f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; visual mesh filename=package://robotiq_description/meshes/visual/robotiq_85_fing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
- added link robotiq_85_right_inner_knuckle_link, mass 0.029951; collision mesh filename=package://robotiq_description/meshes/collision/robotiq_85_i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; visual mesh filename=package://robotiq_description/meshes/visual/robotiq_85_inne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
- added link robotiq_85_right_knuckle_link, mass 0.018491; collision mesh filename=package://robotiq_description/meshes/collision/robotiq_85_k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; visual mesh filename=package://robotiq_description/meshes/visual/robotiq_85_knuc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
- added link robotiq_coupler, mass 0.168; collision mesh filename=package://robotiq_description/meshes/robotiq_85_coupler.stl; visual mesh filename=package://robotiq_description/meshes/robotiq_85_coupler.stl
Joints:
- added joint robotiq_85_base_joint: type fixed, parent robotiq_coupler, child robotiq_85_base_link, origin xyz=0 0 0.004 rpy=0 -1.5707963267948966 3.141592653589793
- added joint robotiq_85_left_finger_joint: type fixed, parent robotiq_85_left_knuckle_link, child robotiq_85_left_finger_link, origin xyz=-0.00408552455 -0.03148604435 0.0 rpy=0 0 0
- added joint robotiq_85_left_finger_tip_joint: type continuous, parent robotiq_85_left_inner_knuckle_link, child robotiq_85_left_finger_tip_link, origin xyz=0.04303959807 -0.03759940821 0.0 rpy=0.0 0.0 0.0, axis 0 0 1, limit lower=-3.14 upper=3.14 effort=0.1 velocity=100.0, mimic joint=robotiq_85_left_knuckle_joint multiplier=-1
- added joint robotiq_85_left_inner_knuckle_joint: type continuous, parent robotiq_85_base_link, child robotiq_85_left_inner_knuckle_link, origin xyz=0.06142 0.0127 0 rpy=3.141592653589793 0.0 0.0, axis 0 0 1, limit lower=-3.14 upper=3.14 effort=0.1 velocity=100.0, mimic joint=robotiq_85_left_knuckle_joint offset=0
- added joint robotiq_85_left_knuckle_joint: type revolute, parent robotiq_85_base_link, child robotiq_85_left_knuckle_link, origin xyz=0.05490451627 0.03060114443 0.0 rpy=3.141592653589793 0.0 0.0, axis 0 0 1, limit lower=0.0 upper=0.80285 effort=1000 velocity=0.5
- added joint robotiq_85_right_finger_joint: type fixed, parent robotiq_85_right_knuckle_link, child robotiq_85_right_finger_link, origin xyz=-0.00408552455 -0.03148604435 0.0 rpy=0 0 0
- added joint robotiq_85_right_finger_tip_joint: type continuous, parent robotiq_85_right_inner_knuckle_link, child robotiq_85_right_finger_tip_link, origin xyz=0.04303959807 -0.03759940821  0.0 rpy=0.0 0.0 0.0, axis 0 0 1, limit lower=-3.14 upper=3.14 effort=0.1 velocity=100.0, mimic joint=robotiq_85_left_knuckle_joint multiplier=-1
- added joint robotiq_85_right_inner_knuckle_joint: type continuous, parent robotiq_85_base_link, child robotiq_85_right_inner_knuckle_link, origin xyz=0.06142 -0.0127 0 rpy=0 0 0, axis 0 0 1, limit lower=-3.14 upper=3.14 effort=0.1 velocity=100.0, mimic joint=robotiq_85_left_knuckle_joint offset=0
- added joint robotiq_85_right_knuckle_joint: type continuous, parent robotiq_85_base_link, child robotiq_85_right_knuckle_link, origin xyz=0.05490451627 -0.03060114443 0.0 rpy=0.0 0.0 0.0, axis 0 0 1, limit lower=-3.14 upper=3.14 effort=1000 velocity=100.0, mimic joint=robotiq_85_left_knuckle_joint
- added joint robotiq_coupler_joint: type fixed, parent ur_tool0, child robotiq_coupler, origin xyz=0 0 0.017 rpy=0 0 -1.5707963267948966

File: robotiq_description/urdf/robotiq_85_gripper.urdf.xacro (robot description, xacro)
@@ -251,5 +251,5 @@
       <minDepth>0.001</minDepth>
     </gazebo>
-    <xacro:robotiq_85_gripper_transmission prefix="${prefix}" />
+    <!-- <xacro:robotiq_85_gripper_transmission prefix="${prefix}" /> -->
   </xacro:macro>
 </robot>
